Commit message: Scooping with cylinder_ellipsoid

File: examples/panda/data/models/franka_description/urdf/panda_arm.urdf (robot description, URDF)
Before this commit: robot panda, 9 links, 8 joints
Links:
- link panda_link0: mass 2.92 -> None
- link panda_link1: mass 2.74 -> 4.970684
- link panda_link2: mass 2.74 -> 0.646926
- link panda_link3: mass 2.38 -> 3.228604
- link panda_link4: mass 2.38 -> 3.587895
- link panda_link5: mass 2.74 -> 1.225946
- link panda_link6: mass 1.55 -> 1.666555
- link panda_link7: mass 0.54 -> 7.35522e-01
- link panda_link8: mass None -> 0.73
